Commit message: z axis rotation fix

File: install/descriptions_package/share/descriptions_package/urdf/bot3.urdf.xacro (robot description, xacro)
@@ -1,6 +1,6 @@
 <?xml version="1.0"?>
 <robot name="bot3" xmlns:xacro="http://www.ros.org.wiki/xacro">
-    <xacro:include filename = "$(find descriptions_package)/urdf/bot3_ext_info.xacro"/>
-    <xacro:include filename = "$(find descriptions_package)/urdf/bot3_control.xacro"/>
+    <!-- <xacro:include filename = "$(find descriptions_package)/urdf/bot3_ext_info.xacro"/>
+    <xacro:include filename = "$(find descriptions_package)/urdf/bot3_control.xacro"/> -->
     <link name="base_footprint" />
     <link
@@ -11,12 +11,12 @@
                 rpy="0 0 0" />
             <mass
-                value="1.0" />
-            <inertia
-                ixx="0.001014"
-                ixy="1.4943E-06"
-                ixz="8.6765E-05"
-                iyy="0.0027467"
-                iyz="2.6408E-07"
-                izz="0.0027686" />
+                value="2.0" />
+            <inertia
+                ixx="0.015"
+                ixy="0"
+                ixz="0"
+                iyy="0.0375"
+                iyz="0.0"
+                izz="0.0275" />
         </inertial>
         <visual>
@@ -44,5 +44,5 @@
         </collision>
     </link>
-    <joint name="base_link" type="fixed">
+    <joint name="base_joint" type="fixed">
         <origin
             xyz="0 0 0.21095"
@@ -60,12 +60,12 @@
                 rpy="0 0 0" />
             <mass
-                value="0.035128" />
-            <inertia
-                ixx="1.2599E-05"
-                ixy="6.3601E-12"
-                ixz="-4.9469E-11"
-                iyy="1.8665E-05"
-                iyz="7.863E-12"
-                izz="1.2601E-05" />
+                value="0.1" />
+            <inertia
+                ixx="0.015"
+                ixy="0"
+                ixz="0"
+                iyy="0.0375"
+                iyz="0.0"
+                izz="0.0275" />
         </inertial>
         <visual>
@@ -88,6 +88,5 @@
                 rpy="0 0 0" />
             <geometry>
-                <mesh
-                    filename="package://descriptions_package/meshes/front_left_wheel_link.STL" />
+                <sphere radius="0.03008" />
             </geometry>
         </collision>
@@ -116,12 +115,12 @@
                 rpy="0 0 0" />
             <mass
-                value="0.035128" />
-            <inertia
-                ixx="1.26E-05"
-                ixy="9.8212E-12"
-                ixz="-4.8774E-10"
-                iyy="1.8665E-05"
-                iyz="2.6737E-12"
-                izz="1.26E-05" />
+                value="0.1" />
+            <inertia
+                ixx="0.015"
+                ixy="0"
+                ixz="0"
+                iyy="0.0375"
+                iyz="0.0"
+                izz="0.0275" />
         </inertial>
         <visual>
@@ -144,6 +143,5 @@
                 rpy="0 0 0" />
             <geometry>
-                <mesh
-                    filename="package://descriptions_package/meshes/front_right_wheel_link.STL" />
+                <sphere radius="0.03008" />
             </geometry>
         </collision>
@@ -172,12 +170,12 @@
                 rpy="0 0 0" />
             <mass
-                value="0.035128" />
-            <inertia
-                ixx="1.2599E-05"
-                ixy="6.3601E-12"
-                ixz="-4.9469E-11"
-                iyy="1.8665E-05"
-                iyz="7.863E-12"
-                izz="1.2601E-05" />
+                value="0.1" />
+            <inertia
+                ixx="0.015"
+                ixy="0"
+                ixz="0"
+                iyy="0.0375"
+                iyz="0.0"
+                izz="0.0275" />
         </inertial>
         <visual>
@@ -200,6 +198,5 @@
                 rpy="0 0 0" />
             <geometry>
-                <mesh
-                    filename="package://descriptions_package/meshes/rear_left_wheel_link.STL" />
+                <sphere radius="0.03008" />
             </geometry>
         </collision>
@@ -228,12 +225,12 @@
                 rpy="0 0 0" />
             <mass
-                value="0.035128" />
-            <inertia
-                ixx="1.26E-05"
-                ixy="9.8212E-12"
-                ixz="-4.8774E-10"
-                iyy="1.8665E-05"
-                iyz="2.6737E-12"
-                izz="1.26E-05" />
+                value="0.1" />
+            <inertia
+                ixx="0.015"
+                ixy="0"
+                ixz="0"
+                iyy="0.0375"
+                iyz="0.0"
+                izz="0.0275" />
         </inertial>
         <visual>
@@ -256,6 +253,5 @@
                 rpy="0 0 0" />
             <geometry>
-                <mesh
-                    filename="package://descriptions_package/meshes/rear_right_wheel_link.STL" />
+                <sphere radius="0.03008" />
             </geometry>
         </collision>
@@ -277,3 +273,23 @@
             velocity="10" />
     </joint>
+    <gazebo>
+        <plugin name="skid_steer_drive" filename="libgazebo_ros_diff_drive.so">
+            <num_wheel_pairs>2</num_wheel_pairs>
+            <left_joint>front_left_wheel_joint</left_joint>
+            <right_joint>front_right_wheel_joint</right_joint>
+            <left_joint>rear_left_wheel_joint</left_joint>
+            <right_joint>rear_right_wheel_joint</right_joint>
+            <wheel_separation>0.200</wheel_separation>
+            <wheel_separation>0.200</wheel_separation>
+            <wheel_diameter>0.06016</wheel_diameter>
+            <wheel_diameter>0.06016</wheel_diameter>
+            <max_wheel_torque>100</max_wheel_torque>
+            <max_wheel_acceleration>10.0</max_wheel_acceleration>
+            <odometry_frame>odom</odometry_frame>
+            <robot_base_frame>base_footprint</robot_base_frame>
+            <publish_odom>true</publish_odom>
+            <publish_odom_tf>true</publish_odom_tf>
+            <publish_wheel_tf>true</publish_wheel_tf>
+        </plugin>
+    </gazebo>
 </robot>

File: install/descriptions_package/share/descriptions_package/urdf/bot3_ext_info.xacro (robot description, xacro)
@@ -1,5 +1,5 @@
 <?xml version="1.0"?>
 <robot name="bot3" xmlns:xacro="http://www.ros.org/wiki/xacro">
-    <transmission name="wheel_front_left_transmission">
+    <!-- <transmission name="wheel_front_left_transmission">
         <plugin>transmission_interface/SimpleTransmission</plugin>
         <actuators name="front_left_wheel_motor" role = "actuator_front_left"/>
@@ -28,9 +28,9 @@
             <mechanical_reduction>1.0</mechanical_reduction>
         </joint>
-    </transmission>
-    <!-- <gazebo reference = "front_left_wheel_link">
-        <mu1>1000000000000000000.0</mu1>
-        <mu2>1000000000000000000.0</mu2>
-        <kp>10000000000.0</kp>
+    </transmission> -->
+    <gazebo reference = "front_left_wheel_link">
+        <mu1>100000000000000.0</mu1>
+        <mu2>100000000000000.0</mu2>
+        <kp>1000000000000.0</kp>
         <kd>10.0</kd>
         <minDepth>0.001</minDepth>
@@ -39,7 +39,7 @@
     </gazebo>
     <gazebo reference = "front_right_wheel_link">
-        <mu1>1000000000000000000.0</mu1>
-        <mu2>1000000000000000000.0</mu2>
-        <kp>10000000000.0</kp>
+        <mu1>100000000000000.0</mu1>
+        <mu2>100000000000000.0</mu2>
+        <kp>1000000000000.0</kp>
         <kd>10.0</kd>
         <minDepth>0.001</minDepth>
@@ -48,7 +48,7 @@
     </gazebo>
     <gazebo reference = "rear_left_wheel_link">
-        <mu1>1000000000000000000.0</mu1>
-        <mu2>1000000000000000000.0</mu2>
-        <kp>10000000000.0</kp>
+        <mu1>100000000000000.0</mu1>
+        <mu2>100000000000000.0</mu2>
+        <kp>1000000000000.0</kp>
         <kd>10.0</kd>
         <minDepth>0.001</minDepth>
@@ -57,12 +57,12 @@
     </gazebo>
     <gazebo reference = "rear_right_wheel_link">
-        <mu1>1000000000000000000.0</mu1>
-        <mu2>1000000000000000000.0</mu2>
-        <kp>10000000000.0</kp>
+        <mu1>100000000000000.0</mu1>
+        <mu2>100000000000000.0</mu2>
+        <kp>1000000000000.0</kp>
         <kd>10.0</kd>
         <minDepth>0.001</minDepth>
         <maxVel>0.1</maxVel>
         <fdir1>1 0 0</fdir1>
-    </gazebo> -->
+    </gazebo>
     <gazebo>
         <plugin filename = "libgazebo_ros2_control.so" name = "gazebo_ros2_control">

Commit message: introduced world

File: install/descriptions_package/share/descriptions_package/urdf/bot3.urdf.xacro (robot description, xacro)
@@ -272,4 +272,62 @@
             effort="100"
             velocity="10" />
+    </joint>
+    <link name="lidar_plate">
+        <inertial>
+            <origin xyz="-7.97972798949331E-17 -2.77555756156289E-17 -0.0015" rpy="0 0 0" />
+            <mass value="0.130589232495131" />
+            <inertia ixx="0.000244952752852722" ixy="-2.05838477476482E-19" ixz="3.17637355220363E-21" iyy="0.000916562838264241" iyz="-3.57552883056295E-21" izz="0.00116131970726822" />
+        </inertial>
+        <visual>
+            <origin xyz="0 0 0" rpy="0 0 0" />
+            <geometry>
+                <mesh filename="package://descriptions_package/meshes/lidar_plate.STL" />
+            </geometry>
+            <material name="">
+                <color rgba="0.792156862745098 0.819607843137255 0.933333333333333 1" />
+            </material>
+        </visual>
+        <collision>
+            <origin xyz="0 0 0" rpy="0 0 0" />
+            <geometry>
+                <mesh filename="package://descriptions_package/meshes/lidar_plate.STL" />
+            </geometry>
+        </collision>
+    </link>
+    <joint name="lidar_plate_joint" type="fixed">
+        <origin xyz="0.0030144 0 0.003" rpy="0 0 0" />
+        <parent link="base_link" />
+        <child link="lidar_plate" />
+        <axis xyz="0 0 0" />
+    </joint>
+    <link name="lidar_sensor">
+        <inertial>
+            <origin xyz="-0.011945780406062 -0.000381929217680526 -0.0170649378129477" rpy="0 0 0" />
+            <mass value="0.073084435549317" />
+            <inertia ixx="1.96074931730795E-05" ixy="-3.62091076640009E-07" ixz="4.28230084046735E-07"
+                     iyy="2.40983835136327E-05" iyz="1.50180909250652E-08"
+                     izz="4.14184164228595E-05" />
+        </inertial>
+        <visual>
+            <origin xyz="0 0 0" rpy="0 0 0" />
+            <geometry>
+                <mesh filename="package://descriptions_package/meshes/laser_link.STL" />
+            </geometry>
+            <material name="">
+                <color rgba="0.298039215686275 0.298039215686275 0.298039215686275 1" />
+            </material>
+        </visual>
+        <collision>
+            <origin xyz="0 0 0" rpy="0 0 0" />
+            <geometry>
+                <mesh filename="package://descriptions_package/meshes/lidar.STL" />
+            </geometry>
+        </collision>
+    </link>
+    <joint name="lidar_joint" type="fixed">
+        <origin xyz="0 0 0.045" rpy="0 0 0" />
+        <parent link="base_link" />
+        <child link="lidar_sensor" />
+        <axis xyz="0 0 0" />
     </joint>
     <gazebo>

Commit message: final commit for SLAM

File: install/descriptions_package/share/descriptions_package/urdf/bot3.urdf.xacro (robot description, xacro)
@@ -326,5 +326,5 @@
     </link>
     <joint name="lidar_joint" type="fixed">
-        <origin xyz="0 0 0.045" rpy="0 0 0" />
+        <origin xyz="0 0 0.045" rpy="0 0 3.14" />
         <parent link="base_link" />
         <child link="lidar_sensor" />
@@ -338,6 +338,6 @@
             <left_joint>rear_left_wheel_joint</left_joint>
             <right_joint>rear_right_wheel_joint</right_joint>
-            <wheel_separation>0.200</wheel_separation>
-            <wheel_separation>0.200</wheel_separation>
+            <wheel_separation>0.190</wheel_separation>
+            <wheel_separation>0.180</wheel_separation>
             <wheel_diameter>0.06016</wheel_diameter>
             <wheel_diameter>0.06016</wheel_diameter>
