Commit message: copied content from workspace_dev , creation of branch under ign-gazebo ros2_control, integrated with mux,slam,nav

File: src/descriptions_package/urdf/bot3.urdf.xacro (robot description, xacro)
@@ -1,4 +1,6 @@
 <?xml version="1.0"?>
 <robot name="bot3" xmlns:xacro="http://www.ros.org.wiki/xacro">
+    <xacro:arg name="is_ignition" default="true"/>
+    <xacro:arg name="is_sim" default="true"/>
     <xacro:include filename = "$(find descriptions_package)/urdf/bot3_ext_info.xacro"/>
     <xacro:include filename = "$(find descriptions_package)/urdf/bot3_control.xacro"/>
@@ -11,12 +13,12 @@
                 rpy="0 0 0" />
             <mass
-                value="10.0" />
-            <inertia
-                ixx="0.015"
-                ixy="0"
-                ixz="0"
-                iyy="0.0375"
-                iyz="0.0"
-                izz="0.0275" />
+                value="8.0" />
+            <inertia
+                ixx="0.016"
+                ixy="0"
+                ixz="0"
+                iyy="0.016"
+                iyz="0.0"
+                izz="0.0185" />
         </inertial>
         <visual>
@@ -60,12 +62,12 @@
                 rpy="0 0 0" />
             <mass
-                value="0.1" />
-            <inertia
-                ixx="0.015"
-                ixy="0"
-                ixz="0"
-                iyy="0.0375"
-                iyz="0.0"
-                izz="0.0275" />
+                value="2.5" />
+            <inertia
+                ixx="0.0015"
+                ixy="0"
+                ixz="0"
+                iyy="0.0015"
+                iyz="0.0"
+                izz="0.00175" />
         </inertial>
         <visual>
@@ -115,12 +117,12 @@
                 rpy="0 0 0" />
             <mass
-                value="0.1" />
-            <inertia
-                ixx="0.015"
-                ixy="0"
-                ixz="0"
-                iyy="0.0375"
-                iyz="0.0"
-                izz="0.0275" />
+                value="2.5" />
+            <inertia
+                ixx="0.0015"
+                ixy="0"
+                ixz="0"
+                iyy="0.0015"
+                iyz="0.0"
+                izz="0.00175" />
         </inertial>
         <visual>
@@ -170,12 +172,12 @@
                 rpy="0 0 0" />
             <mass
-                value="0.1" />
-            <inertia
-                ixx="0.015"
-                ixy="0"
-                ixz="0"
-                iyy="0.0375"
-                iyz="0.0"
-                izz="0.0275" />
+                value="2.5" />
+            <inertia
+                ixx="0.0015"
+                ixy="0"
+                ixz="0"
+                iyy="0.0015"
+                iyz="0.0"
+                izz="0.00175" />
         </inertial>
         <visual>
@@ -225,12 +227,12 @@
                 rpy="0 0 0" />
             <mass
-                value="0.1" />
-            <inertia
-                ixx="0.015"
-                ixy="0"
-                ixz="0"
-                iyy="0.0375"
-                iyz="0.0"
-                izz="0.0275" />
+                value="2.5" />
+            <inertia
+                ixx="0.0015"
+                ixy="0"
+                ixz="0"
+                iyy="0.0015"
+                iyz="0.0"
+                izz="0.00175" />
         </inertial>
         <visual>
@@ -301,5 +303,5 @@
         <axis xyz="0 0 0" />
     </joint>
-    <link name="lidar_sensor">
+    <link name="lidar_sensor_link">
         <inertial>
             <origin xyz="-0.011945780406062 -0.000381929217680526 -0.0170649378129477" rpy="0 0 0" />
@@ -325,29 +327,9 @@
         </collision>
     </link>
-    <joint name="lidar_joint" type="fixed">
+    <joint name="lidar_sensor_joint" type="fixed">
         <origin xyz="0 0 0.045" rpy="0 0 3.14" />
         <parent link="base_link" />
-        <child link="lidar_sensor" />
+        <child link="lidar_sensor_link" />
         <axis xyz="0 0 0" />
     </joint>
-    <gazebo>
-        <plugin name="skid_steer_drive" filename="libgazebo_ros_diff_drive.so">
-            <num_wheel_pairs>2</num_wheel_pairs>
-            <left_joint>front_left_wheel_joint</left_joint>
-            <right_joint>front_right_wheel_joint</right_joint>
-            <left_joint>rear_left_wheel_joint</left_joint>
-            <right_joint>rear_right_wheel_joint</right_joint>
-            <wheel_separation>0.190</wheel_separation>
-            <wheel_separation>0.180</wheel_separation>
-            <wheel_diameter>0.06016</wheel_diameter>
-            <wheel_diameter>0.06016</wheel_diameter>
-            <max_wheel_torque>100</max_wheel_torque>
-            <max_wheel_acceleration>1.0</max_wheel_acceleration>
-            <odometry_frame>odom</odometry_frame>
-            <robot_base_frame>base_footprint</robot_base_frame>
-            <publish_odom>true</publish_odom>
-            <publish_odom_tf>true</publish_odom_tf>
-            <publish_wheel_tf>true</publish_wheel_tf>
-        </plugin>
-    </gazebo>
 </robot>

File: src/descriptions_package/urdf/bot3_control.xacro (robot description, xacro)
@@ -1,12 +1,27 @@
 <?xml version="1.0"?>
 <robot name ="bot3" xmlns:xacro="http://www.ros.org/wiki/xacro">
-    <ros2_control type="system" name="robot_system">
-        <hardware>
-            <plugin>gazebo_ros2_control/GazeboSystem</plugin>
-        </hardware>
+    <ros2_control type="system" name="RobotSystem">
+        <xacro:if value="$(arg is_sim)">
+            <xacro:if value="$(arg is_ignition)">
+                <hardware>
+                    <plugin>ign_ros2_control/IgnitionSystem</plugin>
+                </hardware>
+            </xacro:if>
+            <xacro:unless value="$(arg is_ignition)">
+                <hardware>
+                    <plugin>gz_ros2_control/GazeboSimSystem</plugin>
+                </hardware>
+            </xacro:unless>
+        </xacro:if>
+        <xacro:unless value="$(arg is_sim)">
+            <hardware>
+                <plugin>bot3_firmware/bot_three_interface</plugin>
+                <param name="port">/dev/ttyACM0</param>
+            </hardware>
+        </xacro:unless>
         <joint name="front_left_wheel_joint">
             <command_interface name = "velocity">
-                <param name ="min">-5</param>
-                <param name ="max">5</param>
+                <param name ="min">-10</param>
+                <param name ="max">10</param>
             </command_interface>
             <state_interface name ="position"/>
@@ -15,6 +30,6 @@
         <joint name="front_right_wheel_joint">
             <command_interface name = "velocity">
-                <param name ="min">-5</param>
-                <param name ="max">5</param>
+                <param name ="min">-10</param>
+                <param name ="max">10</param>
             </command_interface>
             <state_interface name ="position"/>
@@ -23,6 +38,6 @@
         <joint name="rear_left_wheel_joint">
             <command_interface name = "velocity">
-                <param name ="min">-5</param>
-                <param name ="max">5</param>
+                <param name ="min">-10</param>
+                <param name ="max">10</param>
             </command_interface>
             <state_interface name ="position"/>
@@ -31,6 +46,6 @@
         <joint name="rear_right_wheel_joint">
             <command_interface name = "velocity">
-                <param name ="min">-5</param>
-                <param name ="max">5</param>
+                <param name ="min">-10</param>
+                <param name ="max">10</param>
             </command_interface>
             <state_interface name ="position"/>

File: src/descriptions_package/urdf/bot3_ext_info.xacro (robot description, xacro)
@@ -30,43 +30,110 @@
     </transmission>
     <gazebo reference = "front_left_wheel_link">
-        <mu1>1000000000000.0</mu1>
-        <mu2>1000000000000.0</mu2>
+        <mu>1.0</mu>
+        <mu2>0.25</mu2>
         <slip1>0.035</slip1>
         <slip2>0</slip2>
-        <fdir1>0 1 0</fdir1>
+        <fdir1>0 0 1</fdir1>
     </gazebo>
     <gazebo reference = "front_right_wheel_link">
-        <mu1>1000000000000.0</mu1>
-        <mu2>1000000000000.0</mu2>
+        <mu>1.0</mu>
+        <mu2>0.25</mu2>
         <slip1>0.035</slip1>
         <slip2>0</slip2>
-        <fdir1>0 1 0</fdir1>
+        <fdir1>0 0 1</fdir1>
     </gazebo>
     <gazebo reference = "rear_left_wheel_link">
-        <mu1>1000000000000.0</mu1>
-        <mu2>1000000000000.0</mu2>
+        <mu>1.0</mu>
+        <mu2>0.25</mu2>
         <slip1>0.035</slip1>
         <slip2>0</slip2>
-        <fdir1>0 1 0</fdir1>
+        <fdir1>0 0 1</fdir1>
     </gazebo>
     <gazebo reference = "rear_right_wheel_link">
-        <mu1>1000000000000.0</mu1>
-        <mu2>1000000000000.0</mu2>
+        <mu>1.0</mu>
+        <mu2>0.25</mu2>
         <slip1>0.035</slip1>
         <slip2>0</slip2>
-        <fdir1>0 1 0</fdir1>
+        <fdir1>0 0 1</fdir1>
     </gazebo>
-    <!-- <gazebo>
-        <plugin filename = "libgazebo_ros2_control.so" name = "gazebo_ros2_control">
-            <robot_param>robot_description</robot_param>
-            <robot_param_node>robot_state_publisher</robot_param_node>
-            <parameters>$(find bot3_controllers)/config/bot3_controller.yaml</parameters>
-        </plugin>
+    <gazebo>
+        <xacro:if value="$(arg is_ignition)">
+            <plugin filename="ign_ros2_control-system" name="ign_ros2_control::IgnitionROS2ControlPlugin">
+                <parameters>$(find bot3_controllers)/config/bot3_controller.yaml</parameters>
+            </plugin>
+            <!-- <plugin filename="ignition-gazebo-imu-system" name= "ignition::gazebo::systems::Imu">
+            </plugin> -->
+            <plugin filename="ignition-gazebo-sensors-system" name="ignition::gazebo::systems::Sensors">
+                <render_engine>ogre2</render_engine>
+            </plugin>
+        </xacro:if>
+        <xacro:unless value="$(arg is_ignition)">
+            <plugin filename="gz_ros2_control-system" name="gz_ros2_control::GazeboSimROS2ControlPlugin">
+                <parameters>$(find bot3_controllers)/config/bot3_controller.yaml</parameters>
+            </plugin>
+            <!-- <plugin filename="gz-sim-imu-system" name="gz::sim::systems::Imu">
+            </plugin> -->
+            <plugin filename="gz-sim-sensors-system" name="gz::sim::systems::Sensors">
+                <render_engine>ogre2</render_engine>
+            </plugin>
+        </xacro:unless>
+    </gazebo>
+    <!-- <gazebo reference="imu_link">
+        <sensor name="imu" type="imu">
+            <always_on>true</always_on>
+            <update_rate>100</update_rate>
+            <gz_frame_id>imu_link</gz_frame_id>
+            <topic>imu</topic>
+            <imu>
+                <angular_velocity>
+                    <x>
+                        <noise type ="gaussian">
+                            <mean>0.0</mean>
+                            <stddev>2e-4</stddev>
+                        </noise>
+                    </x>
+                    <y>
+                        <noise type ="gaussian">
+                            <mean>0.0</mean>
+                            <stddev>2e-4</stddev>
+                        </noise>
+                    </y>
+                    <z>
+                        <noise type ="gaussian">
+                            <mean>0.0</mean>
+                            <stddev>2e-4</stddev>
+                        </noise>
+                    </z>
+                </angular_velocity>
+                <linear_accleration>
+                    <x>
+                        <noise type ="gaussian">
+                            <mean>0.0</mean>
+                            <stddev>1.7e-2</stddev>
+                        </noise>
+                    </x>
+                    <y>
+                        <noise type ="gaussian">
+                            <mean>0.0</mean>
+                            <stddev>1.7e-2</stddev>
+                        </noise>
+                    </y>
+                    <z>
+                        <noise type ="gaussian">
+                            <mean>0.0</mean>
+                            <stddev>1.7e-2</stddev>
+                        </noise>
+                    </z>
+                </linear_accleration>
+            </imu>
+        </sensor>
     </gazebo> -->
-    <gazebo reference="lidar_sensor">
-        <sensor name="rplidar" type ="ray">
+    <gazebo reference="lidar_sensor_link">
+        <sensor name ="lidar" type="gpu_ray">
             <always_on>true</always_on>
             <visualize>true</visualize>
-            <update_rate>10</update_rate>
+            <topic>scan</topic>
+            <update_rate>5</update_rate>
+            <gz_frame_id>lidar_sensor_link</gz_frame_id>
             <ray>
                 <scan>
@@ -74,12 +141,12 @@
                         <samples>360</samples>
                         <resolution>1.0</resolution>
-                        <min_angle>-3.14</min_angle>
-                        <max_angle>3.14</max_angle>
+                        <min_angle>0.0</min_angle>
+                        <max_angle>6.28</max_angle>
                     </horizontal>
                 </scan>
                 <range>
-                    <min>0.12</min>
-                    <max>12.0</max>
-                    <resolution>0.015</resolution>
+                    <min>0.20</min>
+                    <max>8.0</max>
+                    <resolution>0.02</resolution>
                 </range>
                 <noise>
@@ -89,11 +156,4 @@
                 </noise>
             </ray>
-            <plugin name="scan" filename="libgazebo_ros_ray_sensor.so">
-                <ros>
-                    <remapping>~/out:=scan</remapping>
-                </ros>
-                <output_type>sensor_msgs/LaserScan</output_type>
-                <frame_name>lidar_sensor</frame_name>
-            </plugin>
         </sensor>
     </gazebo>
