Commit message: real robot branch commit

File: src/descriptions_package/urdf/bot3.urdf.xacro (robot description, xacro)
@@ -1,4 +1,6 @@
 <?xml version="1.0"?>
 <robot name="bot3" xmlns:xacro="http://www.ros.org.wiki/xacro">
+    <xacro:arg name="is_ignition" default="true"/>
+    <xacro:arg name="is_sim" default="true"/>
     <xacro:include filename = "$(find descriptions_package)/urdf/bot3_ext_info.xacro"/>
     <xacro:include filename = "$(find descriptions_package)/urdf/bot3_control.xacro"/>
@@ -11,12 +13,12 @@
                 rpy="0 0 0" />
             <mass
-                value="10.0" />
-            <inertia
-                ixx="0.015"
-                ixy="0"
-                ixz="0"
-                iyy="0.0375"
-                iyz="0.0"
-                izz="0.0275" />
+                value="8.0" />
+            <inertia
+                ixx="0.016"
+                ixy="0"
+                ixz="0"
+                iyy="0.016"
+                iyz="0.0"
+                izz="0.0185" />
         </inertial>
         <visual>
@@ -60,12 +62,12 @@
                 rpy="0 0 0" />
             <mass
-                value="0.1" />
-            <inertia
-                ixx="0.015"
-                ixy="0"
-                ixz="0"
-                iyy="0.0375"
-                iyz="0.0"
-                izz="0.0275" />
+                value="2.5" />
+            <inertia
+                ixx="0.0015"
+                ixy="0"
+                ixz="0"
+                iyy="0.0015"
+                iyz="0.0"
+                izz="0.00175" />
         </inertial>
         <visual>
@@ -77,9 +79,9 @@
                     filename="package://descriptions_package/meshes/front_left_wheel_link.STL" />
             </geometry>
-            <material
-                name="">
-                <color
-                    rgba="0.29804 0.29804 0.29804 1" />
-            </material>
+<material
+    name="blue material">
+    <color
+        rgba="0.0 0.0 1.0 1" />
+</material>
         </visual>
         <collision>
@@ -115,12 +117,12 @@
                 rpy="0 0 0" />
             <mass
-                value="0.1" />
-            <inertia
-                ixx="0.015"
-                ixy="0"
-                ixz="0"
-                iyy="0.0375"
-                iyz="0.0"
-                izz="0.0275" />
+                value="2.5" />
+            <inertia
+                ixx="0.0015"
+                ixy="0"
+                ixz="0"
+                iyy="0.0015"
+                iyz="0.0"
+                izz="0.00175" />
         </inertial>
         <visual>
@@ -133,7 +135,7 @@
             </geometry>
             <material
-                name="">
+                name="blue material">
                 <color
-                    rgba="0.29804 0.29804 0.29804 1" />
+                    rgba="0.0 0.0 1.0 1" />
             </material>
         </visual>
@@ -170,12 +172,12 @@
                 rpy="0 0 0" />
             <mass
-                value="0.1" />
-            <inertia
-                ixx="0.015"
-                ixy="0"
-                ixz="0"
-                iyy="0.0375"
-                iyz="0.0"
-                izz="0.0275" />
+                value="2.5" />
+            <inertia
+                ixx="0.0015"
+                ixy="0"
+                ixz="0"
+                iyy="0.0015"
+                iyz="0.0"
+                izz="0.00175" />
         </inertial>
         <visual>
@@ -188,7 +190,7 @@
             </geometry>
             <material
-                name="">
+                name="blue material">
                 <color
-                    rgba="0.29804 0.29804 0.29804 1" />
+                    rgba="0.0 0.0 1.0 1" />
             </material>
         </visual>
@@ -225,12 +227,12 @@
                 rpy="0 0 0" />
             <mass
-                value="0.1" />
-            <inertia
-                ixx="0.015"
-                ixy="0"
-                ixz="0"
-                iyy="0.0375"
-                iyz="0.0"
-                izz="0.0275" />
+                value="2.5" />
+            <inertia
+                ixx="0.0015"
+                ixy="0"
+                ixz="0"
+                iyy="0.0015"
+                iyz="0.0"
+                izz="0.00175" />
         </inertial>
         <visual>
@@ -243,7 +245,7 @@
             </geometry>
             <material
-                name="">
+                name="blue material">
                 <color
-                    rgba="0.29804 0.29804 0.29804 1" />
+                    rgba="0.0 0.0 1.0 1" />
             </material>
         </visual>
@@ -284,7 +286,9 @@
                 <mesh filename="package://descriptions_package/meshes/lidar_plate.STL" />
             </geometry>
-            <material name="">
-                <color rgba="0.792156862745098 0.819607843137255 0.933333333333333 1" />
-            </material>
+        <material
+            name="blue material">
+            <color
+                rgba="0.0 0.0 1.0 1" />
+        </material>
         </visual>
         <collision>
@@ -301,5 +305,5 @@
         <axis xyz="0 0 0" />
     </joint>
-    <link name="lidar_sensor">
+    <link name="lidar_sensor_link">
         <inertial>
             <origin xyz="-0.011945780406062 -0.000381929217680526 -0.0170649378129477" rpy="0 0 0" />
@@ -325,29 +329,9 @@
         </collision>
     </link>
-    <joint name="lidar_joint" type="fixed">
+    <joint name="lidar_sensor_joint" type="fixed">
         <origin xyz="0 0 0.045" rpy="0 0 3.14" />
         <parent link="base_link" />
-        <child link="lidar_sensor" />
+        <child link="lidar_sensor_link" />
         <axis xyz="0 0 0" />
     </joint>
-    <gazebo>
-        <plugin name="skid_steer_drive" filename="libgazebo_ros_diff_drive.so">
-            <num_wheel_pairs>2</num_wheel_pairs>
-            <left_joint>front_left_wheel_joint</left_joint>
-            <right_joint>front_right_wheel_joint</right_joint>
-            <left_joint>rear_left_wheel_joint</left_joint>
-            <right_joint>rear_right_wheel_joint</right_joint>
-            <wheel_separation>0.190</wheel_separation>
-            <wheel_separation>0.180</wheel_separation>
-            <wheel_diameter>0.06016</wheel_diameter>
-            <wheel_diameter>0.06016</wheel_diameter>
-            <max_wheel_torque>100</max_wheel_torque>
-            <max_wheel_acceleration>1.0</max_wheel_acceleration>
-            <odometry_frame>odom</odometry_frame>
-            <robot_base_frame>base_footprint</robot_base_frame>
-            <publish_odom>true</publish_odom>
-            <publish_odom_tf>true</publish_odom_tf>
-            <publish_wheel_tf>true</publish_wheel_tf>
-        </plugin>
-    </gazebo>
 </robot>

File: src/descriptions_package/urdf/bot3_control.xacro (robot description, xacro)
@@ -1,12 +1,27 @@
 <?xml version="1.0"?>
 <robot name ="bot3" xmlns:xacro="http://www.ros.org/wiki/xacro">
-    <ros2_control type="system" name="robot_system">
-        <hardware>
-            <plugin>gazebo_ros2_control/GazeboSystem</plugin>
-        </hardware>
+    <ros2_control type="system" name="RobotSystem">
+        <xacro:if value="$(arg is_sim)">
+            <xacro:if value="$(arg is_ignition)">
+                <hardware>
+                    <plugin>ign_ros2_control/IgnitionSystem</plugin>
+                </hardware>
+            </xacro:if>
+            <xacro:unless value="$(arg is_ignition)">
+                <hardware>
+                    <plugin>gz_ros2_control/GazeboSimSystem</plugin>
+                </hardware>
+            </xacro:unless>
+        </xacro:if>
+        <xacro:unless value="$(arg is_sim)">
+            <hardware>
+                <plugin>bot3_firmware/PatrolbotInterface</plugin>
+                <param name="port">/dev/ttyACM0</param>
+            </hardware>
+        </xacro:unless>
         <joint name="front_left_wheel_joint">
             <command_interface name = "velocity">
-                <param name ="min">-5</param>
-                <param name ="max">5</param>
+                <param name ="min">-10</param>
+                <param name ="max">10</param>
             </command_interface>
             <state_interface name ="position"/>
@@ -15,6 +30,6 @@
         <joint name="front_right_wheel_joint">
             <command_interface name = "velocity">
-                <param name ="min">-5</param>
-                <param name ="max">5</param>
+                <param name ="min">-10</param>
+                <param name ="max">10</param>
             </command_interface>
             <state_interface name ="position"/>
@@ -23,6 +38,6 @@
         <joint name="rear_left_wheel_joint">
             <command_interface name = "velocity">
-                <param name ="min">-5</param>
-                <param name ="max">5</param>
+                <param name ="min">-10</param>
+                <param name ="max">10</param>
             </command_interface>
             <state_interface name ="position"/>
@@ -31,6 +46,6 @@
         <joint name="rear_right_wheel_joint">
             <command_interface name = "velocity">
-                <param name ="min">-5</param>
-                <param name ="max">5</param>
+                <param name ="min">-10</param>
+                <param name ="max">10</param>
             </command_interface>
             <state_interface name ="position"/>
