Commit message: improved SLAM and rectified navigation

File: src/descriptions_package/urdf/bot3.urdf.xacro (robot description, xacro)
@@ -1,4 +1,5 @@
 <?xml version="1.0"?>
-<robot name="bot3" xmlns:xacro="http://www.ros.org.wiki/xacro">
+<robot name="bot3"
+    xmlns:xacro="http://www.ros.org.wiki/xacro">
     <xacro:arg name="is_ignition" default="true"/>
     <xacro:arg name="is_sim" default="true"/>
@@ -6,278 +7,148 @@
     <xacro:include filename = "$(find descriptions_package)/urdf/bot3_control.xacro"/>
     <link name="base_footprint" />
-    <link
-        name="base_link">
-        <inertial>
-            <origin
-                xyz="0.018226 -2.0781E-05 -0.13643"
-                rpy="0 0 0" />
-            <mass
-                value="8.0" />
-            <inertia
-                ixx="0.016"
-                ixy="0"
-                ixz="0"
-                iyy="0.016"
-                iyz="0.0"
-                izz="0.0185" />
-        </inertial>
-        <visual>
-            <origin
-                xyz="0 0 0"
-                rpy="0 0 0" />
-            <geometry>
-                <mesh
-                    filename="package://descriptions_package/meshes/base_link.STL" />
-            </geometry>
-            <material
-                name="aluminium extrusion 6063">
-                <color
-                    rgba="0.89804 0.91765 0.92941 1" />
-            </material>
-        </visual>
-        <collision>
-            <origin
-                xyz="0 0 0"
-                rpy="0 0 0" />
-            <geometry>
-                <mesh
-                    filename="package://descriptions_package/meshes/base_link.STL" />
+    <link name="base_link">
+        <inertial>
+            <origin xyz="0.030383 -4.727E-05 -0.22722" rpy="0 0 0" />
+            <mass value="2.9248" />
+            <inertia ixx="0.098824" ixy="4.2644E-05" ixz="0.00018005" iyy="0.18173" iyz="-5.5361E-06" izz="0.21491" />
+        </inertial>
+        <visual>
+            <origin xyz="0 0 0" rpy="0 0 0" />
+            <geometry>
+                <mesh filename="package://descriptions_package/meshes/base_link.STL" />
+            </geometry>
+            <material name="">
+                <color rgba="0.79216 0.81961 0.93333 1" />
+            </material>
+        </visual>
+        <collision>
+            <origin xyz="0 0 0" rpy="0 0 0" />
+            <geometry>
+                <mesh filename="package://descriptions_package/meshes/base_link.STL" />
             </geometry>
         </collision>
     </link>
     <joint name="base_joint" type="fixed">
-        <origin
-            xyz="0 0 0.21095"
-            rpy="0 0 0" />
-        <parent
-            link="base_footprint" />
-        <child
-            link="base_link" />
-    </joint>
-    <link
-        name="front_left_wheel_link">
-        <inertial>
-            <origin
-                xyz="-4.4509E-07 -0.015766 -3.0123E-08"
-                rpy="0 0 0" />
-            <mass
-                value="2.5" />
-            <inertia
-                ixx="0.0015"
-                ixy="0"
-                ixz="0"
-                iyy="0.0015"
-                iyz="0.0"
-                izz="0.00175" />
-        </inertial>
-        <visual>
-            <origin
-                xyz="0 0 0"
-                rpy="0 0 0" />
-            <geometry>
-                <mesh
-                    filename="package://descriptions_package/meshes/front_left_wheel_link.STL" />
-            </geometry>
-<material
-    name="blue material">
-    <color
-        rgba="0.0 0.0 1.0 1" />
-</material>
-        </visual>
-        <collision>
-            <origin
-                xyz="0 0 0"
-                rpy="0 0 0" />
-            <geometry>
-                <sphere radius="0.03008" />
-            </geometry>
-        </collision>
-    </link>
-    <joint
-        name="front_left_wheel_joint"
-        type="continuous">
-        <origin
-            xyz="0.20852 0.10925 -0.18091"
-            rpy="0 0 0" />
-        <parent
-            link="base_link" />
-        <child
-            link="front_left_wheel_link" />
-        <axis
-            xyz="0 1 0" />
-        <limit
-            effort="100"
-            velocity="10" />
-    </joint>
-    <link
-        name="front_right_wheel_link">
-        <inertial>
-            <origin
-                xyz="2.0522E-07 0.015766 3.9719E-07"
-                rpy="0 0 0" />
-            <mass
-                value="2.5" />
-            <inertia
-                ixx="0.0015"
-                ixy="0"
-                ixz="0"
-                iyy="0.0015"
-                iyz="0.0"
-                izz="0.00175" />
-        </inertial>
-        <visual>
-            <origin
-                xyz="0 0 0"
-                rpy="0 0 0" />
-            <geometry>
-                <mesh
-                    filename="package://descriptions_package/meshes/front_right_wheel_link.STL" />
-            </geometry>
-            <material
-                name="blue material">
-                <color
-                    rgba="0.0 0.0 1.0 1" />
-            </material>
-        </visual>
-        <collision>
-            <origin
-                xyz="0 0 0"
-                rpy="0 0 0" />
-            <geometry>
-                <sphere radius="0.03008" />
-            </geometry>
-        </collision>
-    </link>
-    <joint
-        name="front_right_wheel_joint"
-        type="continuous">
-        <origin
-            xyz="0.20852 -0.10925 -0.18091"
-            rpy="0 0 0" />
-        <parent
-            link="base_link" />
-        <child
-            link="front_right_wheel_link" />
-        <axis
-            xyz="0 1 0" />
-        <limit
-            effort="100"
-            velocity="10" />
-    </joint>
-    <link
-        name="rear_left_wheel_link">
-        <inertial>
-            <origin
-                xyz="-4.4509E-07 -0.015766 -3.0123E-08"
-                rpy="0 0 0" />
-            <mass
-                value="2.5" />
-            <inertia
-                ixx="0.0015"
-                ixy="0"
-                ixz="0"
-                iyy="0.0015"
-                iyz="0.0"
-                izz="0.00175" />
-        </inertial>
-        <visual>
-            <origin
-                xyz="0 0 0"
-                rpy="0 0 0" />
-            <geometry>
-                <mesh
-                    filename="package://descriptions_package/meshes/rear_left_wheel_link.STL" />
-            </geometry>
-            <material
-                name="blue material">
-                <color
-                    rgba="0.0 0.0 1.0 1" />
-            </material>
-        </visual>
-        <collision>
-            <origin
-                xyz="0 0 0"
-                rpy="0 0 0" />
-            <geometry>
-                <sphere radius="0.03008" />
-            </geometry>
-        </collision>
-    </link>
-    <joint
-        name="rear_left_wheel_joint"
-        type="continuous">
-        <origin
-            xyz="-0.17248 0.10925 -0.18091"
-            rpy="0 0 0" />
-        <parent
-            link="base_link" />
-        <child
-            link="rear_left_wheel_link" />
-        <axis
-            xyz="0 1 0" />
-        <limit
-            effort="100"
-            velocity="10" />
-    </joint>
-    <link
-        name="rear_right_wheel_link">
-        <inertial>
-            <origin
-                xyz="2.0522E-07 0.015766 3.9719E-07"
-                rpy="0 0 0" />
-            <mass
-                value="2.5" />
-            <inertia
-                ixx="0.0015"
-                ixy="0"
-                ixz="0"
-                iyy="0.0015"
-                iyz="0.0"
-                izz="0.00175" />
-        </inertial>
-        <visual>
-            <origin
-                xyz="0 0 0"
-                rpy="0 0 0" />
-            <geometry>
-                <mesh
-                    filename="package://descriptions_package/meshes/rear_right_wheel_link.STL" />
-            </geometry>
-            <material
-                name="blue material">
-                <color
-                    rgba="0.0 0.0 1.0 1" />
-            </material>
-        </visual>
-        <collision>
-            <origin
-                xyz="0 0 0"
-                rpy="0 0 0" />
-            <geometry>
-                <sphere radius="0.03008" />
-            </geometry>
-        </collision>
-    </link>
-    <joint
-        name="rear_right_wheel_joint"
-        type="continuous">
-        <origin
-            xyz="-0.17248 -0.10925 -0.18091"
-            rpy="0 0 0" />
-        <parent
-            link="base_link" />
-        <child
-            link="rear_right_wheel_link" />
-        <axis
-            xyz="0 1 0" />
-        <limit
-            effort="100"
-            velocity="10" />
+        <origin xyz="0 0 0.3670" rpy="0 0 0" />
+        <parent link="base_footprint" />
+        <child link="base_link" />
+    </joint>
+    <link name="front_left_wheel_link">
+        <inertial>
+            <origin xyz="3.5922E-07 0.010504 6.7014E-07" rpy="0 0 0" />
+            <mass value="0.12758" />
+            <inertia ixx="0.00021109" ixy="-3.2632E-10" ixz="2.7231E-10" iyy="0.00033045" iyz="-7.7919E-10" izz="0.00021109" />
+        </inertial>
+        <visual>
+            <origin xyz="0 0 0" rpy="0 0 0" />
+            <geometry>
+                <mesh filename="package://descriptions_package/meshes/front_left_wheel_link.STL" />
+            </geometry>
+            <material name="">
+                <color rgba="0.79216 0.81961 0.93333 1" />
+            </material>
+        </visual>
+        <collision>
+            <origin xyz="0 0 0" rpy="0 0 0" />
+            <geometry>
+                <mesh filename="package://descriptions_package/meshes/front_left_wheel_link.STL" />
+            </geometry>
+        </collision>
+    </link>
+    <joint name="front_left_wheel_joint" type="continuous">
+        <origin xyz="0.34753 0.22161 -0.30152" rpy="0 0 0" />
+        <parent link="base_link" />
+        <child link="front_left_wheel_link" />
+        <axis xyz="0 1 0" />
+    </joint>
+    <link name="front_right_wheel_link">
+        <inertial>
+            <origin xyz="2.3229E-07 -0.010504 7.234E-07" rpy="0 0 0" />
+            <mass value="0.12758" />
+            <inertia ixx="0.00021109" ixy="3.4532E-10" ixz="3.3275E-10" iyy="0.00033045" iyz="7.6097E-10" izz="0.00021109" />
+        </inertial>
+        <visual>
+            <origin xyz="0 0 0" rpy="0 0 0" />
+            <geometry>
+                <mesh filename="package://descriptions_package/meshes/front_right_wheel_link.STL" />
+            </geometry>
+            <material name="">
+                <color rgba="0.79216 0.81961 0.93333 1" />
+            </material>
+        </visual>
+        <collision>
+            <origin xyz="0 0 0" rpy="0 0 0" />
+            <geometry>
+                <mesh filename="package://descriptions_package/meshes/front_right_wheel_link.STL" />
+            </geometry>
+        </collision>
+    </link>
+    <joint name="front_right_wheel_joint" type="continuous">
+        <origin xyz="0.34753 -0.22341 -0.30152" rpy="0 0 0" />
+        <parent link="base_link" />
+        <child link="front_right_wheel_link" />
+        <axis xyz="0 1 0" />
+    </joint>
+    <link name="rear_left_wheel_link">
+        <inertial>
+            <origin xyz="-7.56215798314308E-07 0.0105035826487469 7.64141164510956E-08" rpy="0 0 0" />
+            <mass value="0.127580085395877" />
+            <inertia ixx="0.000211087485723571" ixy="8.30499338431993E-10" ixz="3.60302607726152E-11" iyy="0.000330454424504559" iyz="5.6828474567577E-14" izz="0.000211086643232728" />
+        </inertial>
+        <visual>
+            <origin xyz="0 0 0" rpy="0 0 0" />
+            <geometry>
+                <mesh filename="package://descriptions_package/meshes/rear_left_wheel_link.STL" />
+            </geometry>
+            <material name="">
+                <color rgba="0.792156862745098 0.819607843137255 0.933333333333333 1" />
+            </material>
+        </visual>
+        <collision>
+            <origin xyz="0 0 0" rpy="0 0 0" />
+            <geometry>
+                <mesh filename="package://descriptions_package/meshes/rear_left_wheel_link.STL" />
+            </geometry>
+        </collision>
+    </link>
+    <joint name="rear_left_wheel_joint" type="continuous">
+        <origin xyz="-0.28747 0.22581 -0.30152" rpy="0 0 0" />
+        <parent link="base_link" />
+        <child link="rear_left_wheel_link" />
+        <axis xyz="0 1 0" />
+    </joint>
+    <link name="rear_right_wheel_link">
+        <inertial>
+            <origin xyz="7.5622E-07 -0.010504 7.6414E-08" rpy="0 0 0" />
+            <mass value="0.12758" />
+            <inertia ixx="0.00021109" ixy="8.305E-10" ixz="-3.603E-11" iyy="0.00033045" iyz="-5.6831E-14" izz="0.00021109" />
+        </inertial>
+        <visual>
+            <origin xyz="0 0 0" rpy="0 0 0" />
+            <geometry>
+                <mesh filename="package://descriptions_package/meshes/rear_right_wheel_link.STL" />
+            </geometry>
+            <material name="">
+                <color rgba="0.79216 0.81961 0.93333 1" />
+            </material>
+        </visual>
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
File: src/descriptions_package/urdf/bot3_control.xacro (robot description, xacro)
@@ -22,6 +22,6 @@
         <joint name="front_left_wheel_joint">
             <command_interface name = "velocity">
-                <param name ="min">-10</param>
-                <param name ="max">10</param>
+                <param name ="min">-20</param>
+                <param name ="max">20</param>
             </command_interface>
             <state_interface name ="position"/>
@@ -30,6 +30,6 @@
         <joint name="front_right_wheel_joint">
             <command_interface name = "velocity">
-                <param name ="min">-10</param>
-                <param name ="max">10</param>
+                <param name ="min">-20</param>
+                <param name ="max">20</param>
             </command_interface>
             <state_interface name ="position"/>
@@ -38,6 +38,6 @@
         <joint name="rear_left_wheel_joint">
             <command_interface name = "velocity">
-                <param name ="min">-10</param>
-                <param name ="max">10</param>
+                <param name ="min">-20</param>
+                <param name ="max">20</param>
             </command_interface>
             <state_interface name ="position"/>
@@ -46,6 +46,6 @@
         <joint name="rear_right_wheel_joint">
             <command_interface name = "velocity">
-                <param name ="min">-10</param>
-                <param name ="max">10</param>
+                <param name ="min">-20</param>
+                <param name ="max">20</param>
             </command_interface>
             <state_interface name ="position"/>

File: src/descriptions_package/urdf/bot3_ext_info.xacro (robot description, xacro)
@@ -129,5 +129,5 @@
         </sensor>
     </gazebo> -->
-    <gazebo reference="lidar_sensor_link">
+    <gazebo reference="laser_frame">
         <sensor name ="lidar" type="gpu_ray">
             <always_on>true</always_on>
